File: Power_25V-30A/00-PCB/fet+curr_sens.sch (KiCad schematic (older format))
At the start: 16 parts, among them Q1 IRL7486, Q2 IRL7486, U1 AD8418, U2 UCC27210

Commit message: Multiplied Phase Schematics
Parts:
- C1, C2, C3, C4, C5, C8: symbol device:C_Small -> Power-board_25V-30A-rescue:C_Small-RESCUE-Power-board_25V-30A
- C6, C7: symbol device:CP1_Small -> Power-board_25V-30A-rescue:CP1_Small-RESCUE-Power-board_25V-30A
- Q1, Q2: symbol Mosfet-[JS]:IRL7486 -> Power-board_25V-30A-rescue:IRL7486-RESCUE-Power-board_25V-30A
- R1, R2, R4: symbol device:R_Small -> Power-board_25V-30A-rescue:R_Small-RESCUE-Power-board_25V-30A
- R3: symbol device:R_Shunt -> Power-board_25V-30A-rescue:R_Shunt-RESCUE-Power-board_25V-30A
- U1: renamed from U2; symbol Power-IC-[JS]:UCC27210 -> Power-board_25V-30A-rescue:UCC27210-RESCUE-Power-board_25V-30A; digikey# 296-30017-1-ND -> 296-30017-1-ND
- U2: renamed from U1; symbol linear_2:AD8417 -> Power-board_25V-30A-rescue:AD8417-RESCUE-Power-board_25V-30A
Connections:
- net +VDC: now also Q1.3 (D); no longer Q1.1 (D)
- net GND: now also Q2.2 (S), U1.~ (VSS); no longer Q2.3 (S), U1.7 (Pad), U1.9 (Pad)
- net PWM_High_Fet: now also U1.~ (VSS); no longer U1.5 (HI)
- net PWM_Low_Fet: now also U1.~ (VSS); no longer U1.6 (LI)
- net VAA: now also U1.~ (VSS); no longer U1.1 (VDD)
- net Voltage_Sens_High: now also Q1.2 (S), Q2.3 (D), U1.~ (VSS); no longer Q1.3 (S), Q2.1 (D), U1.4 (HS)
- net at R1.1: now also Q1.1 (G); no longer Q1.2 (G)
- net at R2.1: now also Q2.1 (G); no longer Q2.2 (G)
- net at C2.1: now also U1.~ (VSS); no longer U1.2 (HB)
- net at R1.2: now also U1.~ (VSS); no longer U1.3 (HO)
- net at R2.2: now also U1.~ (VSS); no longer U1.8 (LO)
- net Phase_Current renamed Phase_Current_Out

Commit message: Changed footprints, used new shunt footprints
Parts:
- Q1, Q2: footprint Mosfet-[JS]:DirectFET-Isometric_ME -> Package_DirectFET:DirectFET_ME
- R3: footprint IPC7351-Nominal:RESC1005X40 -> General_smd-[JS]:CSSK0612
- U1: symbol Power-board_25V-30A-rescue:UCC27210-RESCUE-Power-board_25V-30A -> Power-IC-[JS]:UCC27210
Connections:
- net GND: now also U1.7 (Pad), U1.9 (Pad); no longer U1.~ (VSS)
- net PWM_High_Fet: now also U1.5 (HI); no longer U1.~ (VSS)
- net PWM_Low_Fet: now also U1.6 (LI); no longer U1.~ (VSS)
- net VAA: now also U1.1 (VDD); no longer U1.~ (VSS)
- net Voltage_Sens_High: now also U1.4 (HS); no longer U1.~ (VSS)
- net at R2.2: now also U1.8 (LO); no longer U1.~ (VSS)
- net at R1.2: now also U1.3 (HO); no longer U1.~ (VSS)
- net at C2.1: now also U1.2 (HB); no longer U1.~ (VSS)
Changed lines of the file:
@@
 AR Path="/5A1C142D/5A189276" Ref="U4"  Part="1"
 AR Path="/5A1C15B0/5A189276" Ref="U6"  Part="1"
-F 0 "U6" H 7825 4325 50  0000 C CNN
+F 0 "U2" H 7825 4325 50  0000 C CNN
 F 1 "AD8418" H 7825 4200 50  0000 C CNN
 F 2 "Package_SSOP:MSOP-8_3x3mm_P0.65mm" H 7400 3475 50  0001 C CNN
@@
 AR Path="/5A1C142D/5A18C857" Ref="Q3"  Part="1"
 AR Path="/5A1C15B0/5A18C857" Ref="Q5"  Part="1"
-F 0 "Q5" H 6157 2753 70  0000 L CNN
+F 0 "Q1" H 6157 2753 70  0000 L CNN
 F 1 "IRL7486" H 6157 2639 60  0000 L CNN
-F 2 "Mosfet-[JS]:DirectFET-Isometric_ME" H 5800 2800 60  0001 C CNN
+F 2 "Package_DirectFET:DirectFET_ME" H 5800 2800 60  0001 C CNN
 F 3 "https://www.infineon.com/dgdl/Infineon-IRL7486M-DS-v01_00-EN.pdf?fileId=5546d46258fc0bc10158fec7a83a0629" H 6250 3050 60  0001 C CNN
 F 4 "IRL7486MTRPBF" H 6500 2900 60  0001 C CNN "manf#"
@@
 AR Path="/5A1C142D/5A18C973" Ref="Q4"  Part="1"
 AR Path="/5A1C15B0/5A18C973" Ref="Q6"  Part="1"
-F 0 "Q6" H 6157 3553 70  0000 L CNN
+F 0 "Q2" H 6157 3553 70  0000 L CNN
 F 1 "IRL7486" H 6157 3439 60  0000 L CNN
-F 2 "Mosfet-[JS]:DirectFET-Isometric_ME" H 5800 3600 60  0001 C CNN
+F 2 "Package_DirectFET:DirectFET_ME" H 5800 3600 60  0001 C CNN
 F 3 "https://www.infineon.com/dgdl/Infineon-IRL7486M-DS-v01_00-EN.pdf?fileId=5546d46258fc0bc10158fec7a83a0629" H 6250 3850 60  0001 C CNN
 F 4 "IRL7486MTRPBF" H 6500 3700 60  0001 C CNN "manf#"
@@
 Connection ~ 6050 3100
 $Comp
-L Power-board_25V-30A-rescue:UCC27210-RESCUE-Power-board_25V-30A U1
+L Power-IC-[JS]:UCC27210 U1
 U 1 1 5A18D66A
 P 4875 3000
@@
 AR Path="/5A1C142D/5A18D66A" Ref="U3"  Part="1"
 AR Path="/5A1C15B0/5A18D66A" Ref="U5"  Part="1"
-F 0 "U5" H 5125 3525 60  0000 C CNN
+F 0 "U1" H 5125 3525 60  0000 C CNN
 F 1 "UCC27210" H 5150 3400 60  0000 C CNN
 F 2 "Package_SON:Texas_S-PVSON-N8" H 5075 3425 60  0001 C CNN
 F 3 "http://www.ti.com/lit/ds/symlink/ucc27210.pdf" H 5175 3525 60  0001 C CNN
-F 4 "UCC27210DRMT " H 5275 3625 60  0001 C CNN "manf#"
-F 5 "296-30017-1-ND" H 5375 3725 60  0001 C CNN "digikey#"
+F 4 "296-30017-1-ND" H 5375 3725 60  0001 C CNN "digikey#"
+F 5 "UCC27210DRMT " H 5275 3625 60  0001 C CNN "manf#"
 	1    4875 3000
 	1    0    0    -1
@@
 AR Path="/5A1C142D/5A18D7E0" Ref="R6"  Part="1"
 AR Path="/5A1C15B0/5A18D7E0" Ref="R10"  Part="1"
-F 0 "R10" V 5575 3500 50  0000 C CNN
+F 0 "R2" V 5575 3500 50  0000 C CNN
 F 1 "4R7" V 5725 3500 50  0000 C CNN
 F 2 "IPC7351-Nominal:RESC0603X30" H 5650 3500 50  0001 C CNN
@@
 AR Path="/5A1C142D/5A18D9F7" Ref="R5"  Part="1"
 AR Path="/5A1C15B0/5A18D9F7" Ref="R9"  Part="1"
-F 0 "R9" V 5575 2700 50  0000 C CNN
+F 0 "R1" V 5575 2700 50  0000 C CNN
 F 1 "4R7" V 5725 2700 50  0000 C CNN
 F 2 "IPC7351-Nominal:RESC0603X30" H 5650 2700 50  0001 C CNN
@@
 AR Path="/5A1C142D/5A18DDEC" Ref="C10"  Part="1"
 AR Path="/5A1C15B0/5A18DDEC" Ref="C18"  Part="1"
-F 0 "C18" H 5325 2975 50  0000 L CNN
+F 0 "C2" H 5325 2975 50  0000 L CNN
 F 1 "0µF1" H 5325 2825 50  0000 L CNN
 F 2 "IPC7351-Nominal:CAPC0603X33" H 5275 2900 50  0001 C CNN
@@
 AR Path="/5A1C142D/5A18E6B6" Ref="#PWR017"  Part="1"
 AR Path="/5A1C15B0/5A18E6B6" Ref="#PWR029"  Part="1"
-F 0 "#PWR029" H 6050 4150 50  0001 C CNN
+F 0 "#PWR05" H 6050 4150 50  0001 C CNN
 F 1 "GND" H 6055 4227 50  0000 C CNN
 F 2 "" H 6050 4400 50  0001 C CNN
@@
 AR Path="/5A1C142D/5A18EF6A" Ref="#PWR015"  Part="1"
 AR Path="/5A1C15B0/5A18EF6A" Ref="#PWR027"  Part="1"
-F 0 "#PWR027" H 4825 3300 50  0001 C CNN
+F 0 "#PWR03" H 4825 3300 50  0001 C CNN
 F 1 "GND" H 4830 3377 50  0000 C CNN
 F 2 "" H 4825 3550 50  0001 C CNN
@@
 AR Path="/5A1C142D/5A18FE90" Ref="R7"  Part="1"
 AR Path="/5A1C15B0/5A18FE90" Ref="R11"  Part="1"
-F 0 "R11" V 7125 3100 50  0000 C CNN
+F 0 "R3" V 7125 3100 50  0000 C CNN
 F 1 "0R005" V 7216 3100 50  0000 C CNN
-F 2 "IPC7351-Nominal:RESC1005X40" V 7280 3100 50  0001 C CNN
+F 2 "General_smd-[JS]:CSSK0612" V 7280 3100 50  0001 C CNN
 F 3 "" H 7350 3100 50  0001 C CNN
 	1    7350 3100
@@
 AR Path="/5A1C142D/5A191474" Ref="#PWR016"  Part="1"
 AR Path="/5A1C15B0/5A191474" Ref="#PWR028"  Part="1"
-F 0 "#PWR028" H 6050 2100 50  0001 C CNN
+F 0 "#PWR04" H 6050 2100 50  0001 C CNN
 F 1 "+VDC" H 6050 2475 50  0000 C CNN
 F 2 "" H 6050 2200 50  0001 C CNN
@@
 AR Path="/5A1C142D/5A191D2A" Ref="#PWR021"  Part="1"
 AR Path="/5A1C15B0/5A191D2A" Ref="#PWR033"  Part="1"
-F 0 "#PWR033" H 7350 4150 50  0001 C CNN
+F 0 "#PWR09" H 7350 4150 50  0001 C CNN
 F 1 "GND" H 7355 4227 50  0000 C CNN
 F 2 "" H 7350 4400 50  0001 C CNN
@@
 AR Path="/5A1C142D/5A191F32" Ref="#PWR014"  Part="1"
 AR Path="/5A1C15B0/5A191F32" Ref="#PWR026"  Part="1"
-F 0 "#PWR026" H 4825 2050 50  0001 C CNN
+F 0 "#PWR02" H 4825 2050 50  0001 C CNN
 F 1 "VAA" H 4842 2373 50  0000 C CNN
 F 2 "" H 4825 2200 50  0001 C CNN
@@
 AR Path="/5A1C142D/5A19302F" Ref="#PWR018"  Part="1"
 AR Path="/5A1C15B0/5A19302F" Ref="#PWR030"  Part="1"
-F 0 "#PWR030" H 6800 3625 50  0001 C CNN
+F 0 "#PWR06" H 6800 3625 50  0001 C CNN
 F 1 "VAA" H 6817 3948 50  0000 C CNN
 F 2 "" H 6800 3775 50  0001 C CNN
@@
 AR Path="/5A1C142D/5A1942B4" Ref="C11"  Part="1"
 AR Path="/5A1C15B0/5A1942B4" Ref="C19"  Part="1"
-F 0 "C19" H 6850 4250 50  0000 L CNN
+F 0 "C3" H 6850 4250 50  0000 L CNN
 F 1 "2µF2" H 6850 4100 50  0000 L CNN
 F 2 "IPC7351-Nominal:CAPC0603X33" H 6800 4175 50  0001 C CNN
@@
 AR Path="/5A1C142D/5A19740C" Ref="R8"  Part="1"
 AR Path="/5A1C15B0/5A19740C" Ref="R12"  Part="1"
-F 0 "R12" V 7975 3825 50  0000 C CNN
+F 0 "R4" V 7975 3825 50  0000 C CNN
 F 1 "100R" V 8125 3825 50  0000 C CNN
 F 2 "IPC7351-Nominal:RESC0603X30" H 8050 3825 50  0001 C CNN
@@
 AR Path="/5A1C142D/5A1974AE" Ref="C16"  Part="1"
 AR Path="/5A1C15B0/5A1974AE" Ref="C24"  Part="1"
-F 0 "C24" H 8300 4175 50  0000 L CNN
+F 0 "C8" H 8300 4175 50  0000 L CNN
 F 1 "4nF7" H 8300 4025 50  0000 L CNN
 F 2 "IPC7351-Nominal:CAPC0603X33" H 8250 4100 50  0001 C CNN
@@
 AR Path="/5A1C142D/5A197546" Ref="#PWR024"  Part="1"
 AR Path="/5A1C15B0/5A197546" Ref="#PWR036"  Part="1"
-F 0 "#PWR036" H 8250 4150 50  0001 C CNN
+F 0 "#PWR012" H 8250 4150 50  0001 C CNN
 F 1 "GND" H 8255 4227 50  0000 C CNN
 F 2 "" H 8250 4400 50  0001 C CNN
@@
 AR Path="/5A1C142D/5A19E039" Ref="C9"  Part="1"
 AR Path="/5A1C15B0/5A19E039" Ref="C17"  Part="1"
-F 0 "C17" H 4500 2475 50  0000 L CNN
+F 0 "C1" H 4500 2475 50  0000 L CNN
 F 1 "2µF2" H 4500 2325 50  0000 L CNN
 F 2 "IPC7351-Nominal:CAPC0603X33" H 4450 2400 50  0001 C CNN
@@
 AR Path="/5A1C142D/5A19F212" Ref="#PWR013"  Part="1"
 AR Path="/5A1C15B0/5A19F212" Ref="#PWR025"  Part="1"
-F 0 "#PWR025" H 4450 2325 50  0001 C CNN
+F 0 "#PWR01" H 4450 2325 50  0001 C CNN
 F 1 "GND" H 4455 2402 50  0000 C CNN
 F 2 "" H 4450 2575 50  0001 C CNN
@@
 AR Path="/5A1C142D/5A1A101B" Ref="C13"  Part="1"
 AR Path="/5A1C15B0/5A1A101B" Ref="C21"  Part="1"
-F 0 "C21" H 7075 2475 50  0000 L CNN
+F 0 "C5" H 7075 2475 50  0000 L CNN
 F 1 "4nF7" H 7075 2325 50  0000 L CNN
 F 2 "IPC7351-Nominal:CAPC0603X33" H 7025 2400 50  0001 C CNN
@@
 AR Path="/5A1C142D/5A1A10BC" Ref="#PWR019"  Part="1"
 AR Path="/5A1C15B0/5A1A10BC" Ref="#PWR031"  Part="1"
-F 0 "#PWR031" H 6925 2100 50  0001 C CNN
+F 0 "#PWR07" H 6925 2100 50  0001 C CNN
 F 1 "+VDC" H 6925 2475 50  0000 C CNN
 F 2 "" H 6925 2200 50  0001 C CNN
@@
 AR Path="/5A1C142D/5A1A10E1" Ref="C12"  Part="1"
 AR Path="/5A1C15B0/5A1A10E1" Ref="C20"  Part="1"
-F 0 "C20" H 6875 2475 50  0000 L CNN
+F 0 "C4" H 6875 2475 50  0000 L CNN
 F 1 "4nF7" H 6875 2325 50  0000 L CNN
 F 2 "IPC7351-Nominal:CAPC0603X33" H 6825 2400 50  0001 C CNN
@@
 AR Path="/5A1C142D/5A1A1129" Ref="#PWR020"  Part="1"
 AR Path="/5A1C15B0/5A1A1129" Ref="#PWR032"  Part="1"
-F 0 "#PWR032" H 6925 2350 50  0001 C CNN
+F 0 "#PWR08" H 6925 2350 50  0001 C CNN
 F 1 "GND" H 6930 2427 50  0000 C CNN
 F 2 "" H 6925 2600 50  0001 C CNN
@@
 AR Path="/5A1C142D/5A1A7817" Ref="#PWR022"  Part="1"
 AR Path="/5A1C15B0/5A1A7817" Ref="#PWR034"  Part="1"
-F 0 "#PWR034" H 8025 2100 50  0001 C CNN
+F 0 "#PWR010" H 8025 2100 50  0001 C CNN
 F 1 "+VDC" H 8025 2475 50  0000 C CNN
 F 2 "" H 8025 2200 50  0001 C CNN
@@
 AR Path="/5A1C142D/5A1A7823" Ref="#PWR023"  Part="1"
 AR Path="/5A1C15B0/5A1A7823" Ref="#PWR035"  Part="1"
-F 0 "#PWR035" H 8025 2350 50  0001 C CNN
+F 0 "#PWR011" H 8025 2350 50  0001 C CNN
 F 1 "GND" H 8030 2427 50  0000 C CNN
 F 2 "" H 8025 2600 50  0001 C CNN
@@
 AR Path="/5A1C142D/5A1A78FC" Ref="C14"  Part="1"
 AR Path="/5A1C15B0/5A1A78FC" Ref="C22"  Part="1"
-F 0 "C22" H 8016 2446 50  0000 L CNN
+F 0 "C6" H 8016 2446 50  0000 L CNN
 F 1 "680µF_50V" H 8016 2355 50  0000 L CNN
 F 2 "" H 7925 2400 50  0001 C CNN
@@
 AR Path="/5A1C142D/5A1A79DA" Ref="C15"  Part="1"
 AR Path="/5A1C15B0/5A1A79DA" Ref="C23"  Part="1"
-F 0 "C23" H 8216 2446 50  0000 L CNN
+F 0 "C7" H 8216 2446 50  0000 L CNN
 F 1 "680µF_50V" H 8216 2355 50  0000 L CNN
 F 2 "" H 8125 2400 50  0001 C CNN

Commit message: testing arrangements for 3 phase power stage
Parts:
- removed C1: 2µF2, IPC7351-Nominal:CAPC0603X33, symbol Power-board_25V-30A-rescue:C_Small-RESCUE-Power-board_25V-30A
- removed C8: 4nF7, IPC7351-Nominal:CAPC0603X33, symbol Power-board_25V-30A-rescue:C_Small-RESCUE-Power-board_25V-30A
- removed Q1, Q2: IRL7486, Package_DirectFET:DirectFET_ME, symbol Power-board_25V-30A-rescue:IRL7486-RESCUE-Power-board_25V-30A
- removed R3: 0R005, General_smd-[JS]:CSSK0612, symbol Power-board_25V-30A-rescue:R_Shunt-RESCUE-Power-board_25V-30A
- removed R4: 100R, IPC7351-Nominal:RESC0603X30, symbol Power-board_25V-30A-rescue:R_Small-RESCUE-Power-board_25V-30A
- removed U1: UCC27210, Package_SON:Texas_S-PVSON-N8, symbol Power-IC-[JS]:UCC27210
- removed U2: AD8418, Package_SSOP:MSOP-8_3x3mm_P0.65mm, symbol Power-board_25V-30A-rescue:AD8417-RESCUE-Power-board_25V-30A
- added C9: 0µF1, IPC7351-Nominal:CAPC0603X33, symbol Power-board_25V-30A-rescue:C_Small-RESCUE-Power-board_25V-30A
- added Q1, Q2: IRL7486, Mosfet-[JS]:DirectFET_ME, symbol Mosfet-[JS]:IRL7486
- added R3: 0R0005, IPC7351-Nominal:RESC3216X63, symbol device:R_Small
- added U2: UCC27210, Package_SON:Texas_S-PVSON-N8, symbol Power-IC-[JS]:UCC27210
- added U3: LT6118, Package_DFN_QFN:DFN-8-1EP_3x2mm_P0.45mm, symbol Power-IC-[JS]:LT6118
- renumbered C2 to C8, R1 to R2, R2 to R4
Connections:
- net +VDC: now also Q1.1 (D)
- net Current_Sens: now also U3.6 (OUT_An)
- net GND: now also C9.2, Q2.3 (S), U2.7 (Pad), U2.9 (Pad), U3.2 (LE), U3.4 (V-), U3.5 (IN_Comp), U3.9 (PAD)
- net PWM_High_Fet: now also U2.5 (HI)
- net PWM_Low_Fet: now also U2.6 (LI)
- net Phase_Current_Out: now also R3.1, U3.1 (SENSE_LO)
- net Voltage_Sens_High: now also Q1.3 (S), Q2.1 (D), R3.2, U2.4 (HS), U3.8 (SENSE_HI)
- net at R2.1: now also Q1.2 (G)
- net at R4.1: now also Q2.2 (G)
- net at C8.1: now also U2.2 (HB)
- net at R2.2: now also U2.3 (HO)
- net at R4.2: now also U2.8 (LO)
- net VAA renamed VCC
- net VCC: now also C9.1, U2.1 (VDD), U3.7 (V+)
- no-connect marks 0 -> 1
Other:
- moved on the sheet: C8
